File: ai03-pcb-guide.sch (KiCad schematic (older format))
At the start: 24 parts, among them SW1 SW_Push, U1 ATmega32U4-AU, Y1 16MHz

Commit message: Finished PCB traces
Parts:
- renumbered D3 to D2, D2 to D3, MX3 to MX2, MX2 to MX3
Connections:
- net COL0: now also U1.29 (PB5); no longer D1.1 (K), D2.1 (K)
- net COL1: now also U1.28 (PB4)
- net ROW1: now also U1.30 (PB6)
- net ROW0: now reaches U1.27 (PD7)
- net ROW0: now also D1.1 (K), D2.1 (K)
Changed lines of the file:
@@
 EESchema Schematic File Version 4
+LIBS:ai03-pcb-guide-cache
 EELAYER 30 0
 EELAYER END
@@
 $EndDescr
 $Comp
-L MCU_Microchip_ATmega:ATmega32U4-AU U1
-U 1 1 607C8AD4
-P 3250 3800
-F 0 "U1" H 3250 1911 50  0000 C CNN
-F 1 "ATmega32U4-AU" H 3250 1820 50  0000 C CNN
-F 2 "Package_QFP:TQFP-44_10x10mm_P0.8mm" H 3250 3800 50  0001 C CIN
-F 3 "http://ww1.microchip.com/downloads/en/DeviceDoc/Atmel-7766-8-bit-AVR-ATmega16U4-32U4_Datasheet.pdf" H 3250 3800 50  0001 C CNN
-	1    3250 3800
-	1    0    0    -1
-$EndComp
-$Comp
 L power:+5V #PWR0101
 U 1 1 607CA60D
@@
 Wire Wire Line
 	3150 1850 3150 2000
-Wire Wire Line
-	3150 2000 3250 2000
-Connection ~ 3150 2000
-Wire Wire Line
-	3250 2000 3350 2000
-Connection ~ 3250 2000
 $Comp
 L power:GND #PWR0102
@@
 	1    0    0    -1
 $EndComp
-Wire Wire Line
-	3150 5600 3250 5600
-Wire Wire Line
-	3150 5600 2800 5600
-Connection ~ 3150 5600
 $Comp
 L Device:R_Small R4
@@
 	1    0    0    -1
 $EndComp
-Wire Wire Line
-	3850 4400 4450 4400
-Wire Wire Line
-	4650 4400 5200 4400
 $Comp
 L Device:R_Small R2
@@
 $EndComp
 $Comp
-L MX_Alps_Hybrid:MX-NoLED MX3
+L MX_Alps_Hybrid:MX-NoLED MX2
 U 1 1 6082D1FF
 P 7500 3650
-F 0 "MX3" H 7533 3873 60  0000 C CNN
+F 0 "MX2" H 7533 3873 60  0000 C CNN
 F 1 "MX-NoLED" H 7533 3799 20  0000 C CNN
 F 2 "MX_Alps_Hybrid:MX-1U" H 6875 3625 60  0001 C CNN
@@
 	7450 3900 7350 3900
 $Comp
-L Device:D_Small D3
+L Device:D_Small D2
 U 1 1 6082D207
 P 7350 4000
-F 0 "D3" V 7396 3932 50  0000 R CNN
+F 0 "D2" V 7396 3932 50  0000 R CNN
 F 1 "D_Small" V 7305 3932 50  0000 R CNN
 F 2 "Diode_SMD:D_SOD-123" V 7350 4000 50  0001 C CNN
@@
 $EndComp
 $Comp
-L MX_Alps_Hybrid:MX-NoLED MX2
+L MX_Alps_Hybrid:MX-NoLED MX3
 U 1 1 6082F2D2
 P 6800 4500
-F 0 "MX2" H 6833 4723 60  0000 C CNN
+F 0 "MX3" H 6833 4723 60  0000 C CNN
 F 1 "MX-NoLED" H 6833 4649 20  0000 C CNN
 F 2 "MX_Alps_Hybrid:MX-1U" H 6175 4475 60  0001 C CNN
@@
 	6750 4750 6650 4750
 $Comp
-L Device:D_Small D2
+L Device:D_Small D3
 U 1 1 6082F2DA
 P 6650 4850
-F 0 "D2" V 6696 4782 50  0000 R CNN
+F 0 "D3" V 6696 4782 50  0000 R CNN
 F 1 "D_Small" V 6605 4782 50  0000 R CNN
 F 2 "Diode_SMD:D_SOD-123" V 6650 4850 50  0001 C CNN
@@
 $EndComp
 Wire Wire Line
-	6950 3600 6950 4100
-Wire Wire Line
 	6950 4100 6650 4100
 Wire Wire Line
@@
 Wire Wire Line
 	6950 4100 7350 4100
-Connection ~ 6950 4100
 Wire Wire Line
 	7650 3600 7650 3300
@@
 	7650 3600 7650 4450
 Connection ~ 7650 3600
-Wire Wire Line
-	6950 4100 6950 4450
 Wire Wire Line
 	7350 4950 6650 4950
@@
 Text GLabel 7650 3300 1    50   Input ~ 0
 COL1
+Text GLabel 3850 2700 2    50   Input ~ 0
+COL1
+Connection ~ 3150 5600
+Wire Wire Line
+	3150 5600 2800 5600
+Wire Wire Line
+	3150 5600 3250 5600
+Connection ~ 3250 2000
+Connection ~ 3150 2000
+Wire Wire Line
+	3250 2000 3350 2000
+Wire Wire Line
+	3150 2000 3250 2000
+Wire Wire Line
+	4650 4400 5200 4400
+Wire Wire Line
+	3850 4400 4450 4400
+$Comp
+L MCU_Microchip_ATmega:ATmega32U4-AU U1
+U 1 1 607C8AD4
+P 3250 3800
+F 0 "U1" H 3250 1911 50  0000 C CNN
+F 1 "ATmega32U4-AU" H 3250 1820 50  0000 C CNN
+F 2 "Package_QFP:TQFP-44_10x10mm_P0.8mm" H 3250 3800 50  0001 C CIN
+F 3 "http://ww1.microchip.com/downloads/en/DeviceDoc/Atmel-7766-8-bit-AVR-ATmega16U4-32U4_Datasheet.pdf" H 3250 3800 50  0001 C CNN
+	1    3250 3800
+	1    0    0    -1
+$EndComp
+Text GLabel 3850 2800 2    50   Input ~ 0
+COL0
+Text GLabel 3850 2900 2    50   Input ~ 0
+ROW1
 Text GLabel 6300 4100 0    50   Input ~ 0
 ROW0
 Text GLabel 6300 4950 0    50   Input ~ 0
 ROW1
+Text GLabel 3850 4200 2    50   Input ~ 0
+ROW0
+Wire Wire Line
+	6950 3600 6950 4450
 $EndSCHEMATC
