File: ai03-pcb-guide.kicad_pcb (KiCad board)
At the start: 2 copper layers, 79.4 x 38.1 mm, 24 parts, among them SW1 SW_Push, U1 ATmega32U4-AU, Y1 16MHz

Commit message: Finished PCB traces
Parts:
- removed the D3 at (177.8, 127.8)
- added D2: D_Small, Diode_SMD:D_SOD-123, B.Cu at (177.8, 127.8)
- moved C7 6.13 mm to (119.9, 146.1), turned to 270 degrees
- moved C5 1.77 mm to (121.3, 130.7)
- moved R3 1.77 mm to (118.2, 130.7), turned to 270 degrees
- moved F1 1.00 mm to (103.2, 136.5), turned to 90 degrees
- moved C6 0.88 mm to (118.9, 138.9)
- moved R1 0.79 mm to (105.6, 130.3)
- moved R2 0.79 mm to (109.5, 130.3)
- turned SW1 to 180 degrees
- renumbered D2 to D3, MX3 to MX2, MX2 to MX3
Connections:
- D1 pad 1: COL0 -> ROW0
- U1 pad 27: Net-(U1-Pad27) -> ROW0
- U1 pad 28: Net-(U1-Pad28) -> COL1
- U1 pad 29: Net-(U1-Pad29) -> COL0
- U1 pad 30: Net-(U1-Pad30) -> ROW1
Routing:
- net GND: track 0.00 -> 115.8 mm
- net +5V: track 0.00 -> 102.4 mm, vias 0 -> 5
- net COL1: track 0.00 -> 53.7 mm
- net ROW1: track 0.00 -> 52.3 mm
- net ROW0: track 0.00 -> 48.1 mm
- net Net-(R3-Pad2): track 0.00 -> 33.5 mm, vias 0 -> 2
- net COL0: track 0.00 -> 32.7 mm
- net Net-(R1-Pad1): track 0.00 -> 26.0 mm
- net Net-(R2-Pad1): track 0.00 -> 24.8 mm
- net Net-(C4-Pad1): track 0.00 -> 11.9 mm
- net VCC: track 0.00 -> 11.3 mm
- net Net-(C3-Pad1): track 0.00 -> 8.50 mm
- net Net-(D3-Pad2): track 0.00 -> 6.67 mm
- net Net-(D4-Pad2): track 0.00 -> 6.67 mm
- net Net-(D2-Pad2): track 0.00 -> 6.67 mm
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Other:
- net class Default: trace_width 10 -> 0.254
- net class Power: trace_width 15 -> 0.381

Commit message: Finished PCB
Routing:
- added copper zone on B.Cu, net GND
Other:
- board text added: "First PCB Design! - 4/18/2021"
Changed lines of the file:
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@@
   (general
     (thickness 1.6)
-    (drawings 8)
+    (drawings 9)
     (tracks 191)
     (zones 0)
@@
       (rotate (xyz 0 0 0))
     )
+  )
+  (gr_text "First PCB Design!\n- 4/18/2021" (at 122.2375 152.4) (layer B.SilkS)
+    (effects (font (size 1 1) (thickness 0.15)) (justify mirror))
   )
   (gr_line (start 102.39375 118.26875) (end 177.00625 118.26875) (layer Edge.Cuts) (width 0.05))
@@
   (segment (start 150.5375 138.36025) (end 158.75 130.14775) (width 0.254) (layer B.Cu) (net 44))
   (segment (start 135.113 138.36025) (end 150.5375 138.36025) (width 0.254) (layer B.Cu) (net 44))
+  (zone (net 1) (net_name GND) (layer B.Cu) (hatch edge 0.508)
+    (connect_pads (clearance 0.508))
+    (min_thickness 0.254)
+    (fill yes (arc_segments 32) (thermal_gap 0.508) (thermal_bridge_width 0.508))
+    (polygon
+      (pts
+        (xy 141.2875 118.26875) (xy 100.0125 118.26875) (xy 100.0125 156.36875) (xy 141.2875 156.36875)
+      )
+    )
+  )
 )
